File: USBcablecracker.kicad_pcb (KiCad board)
At the start: 2 copper layers, 100 x 50 mm, 53 parts, among them P1 USB_A, P10 USB_A, P11 USB_B, P12 CONN_01X09, P2 CONN_01X02, P3 USB_B-Micro, P6 CONN_01X09, P7 USB_B-Mini, P8 USB_B-Micro-3.0, P9 USB_TYPEC-S, SW1 Switch_SPDT_x2, U1 ATmega32U4-AU, U2 LMV358, U3 AD623, Y1 16MHz

Commit message: update
Parts:
- added C13: 1nF, Capacitors_SMD:C_0603_HandSoldering, B.Cu at (110.7, 84.0)
- added R20: 10K, Resistors_SMD:R_0603_HandSoldering, B.Cu at (123.1, 87.0)
- added R21: 10K, Resistors_SMD:R_0603_HandSoldering, B.Cu at (111.3, 79.9)
- added R22: 10K, Resistors_SMD:R_0603_HandSoldering, B.Cu at (109.8, 76.7)
- R11: value 1K -> 10K
- R12: value 1K -> 100K
- R13: value 100K -> 10K
- R17: value 220 -> 68
- R18: value 150 -> 33
- R19: value 10k -> 11k
- moved R11 8.62 mm to (107.8, 84.8)
- moved R13 7.31 mm to (106.3, 88.2), turned to 90 degrees
- moved C2 6.30 mm to (112.1, 86.8), turned to 270 degrees
- moved R12 5.20 mm to (107.8, 82.9), turned to 0 degrees
- moved P8 0.82 mm to (104.8, 96.2)
- turned R17 to 180 degrees
Connections:
- C10 pad 2: +5V -> +5C
- C11 pad 2: +5V -> +5C
- C12 pad 2: +5V -> +5C
- C2 pad 1: Net-(C2-Pad1) -> Net-(C13-Pad1)
- C2 pad 2: GND -> Net-(C2-Pad2)
- C3 pad 2: Net-(C3-Pad2) -> Net-(C2-Pad2)
- C8 pad 1: +5V -> +5C
- C9 pad 2: +5V -> +5C
- CONN1 pad 2: +5V -> +5C
- D1 pad 2: +5V -> +5C
- D2 pad 2: +5V -> +5C
- DS1 pad 15: +5V -> +5C
- DS1 pad 2: +5V -> +5C
- P3 pad 1: +5V -> +5C
- P6 pad 1: +5V -> +5C
- R1 pad 1: +5V -> +5C
- R11 pad 1: /REFO -> Net-(C13-Pad1)
- R11 pad 2: Net-(C2-Pad1) -> /TP2
- R12 pad 1: Net-(C2-Pad1) -> Net-(C13-Pad1)
- R12 pad 2: GND -> /REFO
- R13 pad 1: Net-(C3-Pad2) -> Net-(C2-Pad2)
- R13 pad 2: Net-(C2-Pad1) -> /TP1
- R14 pad 2: Net-(C3-Pad2) -> Net-(C2-Pad2)
- R17 pad 1: /TP1 -> /REFO
- R17 pad 2: Net-(C3-Pad1) -> /TP1
- R5 pad 2: +5V -> +5C
- R9 pad 2: +5V -> +5C
- U1 pad 14: +5V -> +5C
- U1 pad 2: +5V -> +5C
- U1 pad 24: +5V -> +5C
- U1 pad 34: +5V -> +5C
- U1 pad 44: +5V -> +5C
- U2 pad 2: Net-(C3-Pad2) -> Net-(C2-Pad2)
- U2 pad 3: /REFO -> Net-(C13-Pad1)
- U2 pad 6: /REFO -> Net-(R20-Pad2)
- U2 pad 8: +5V -> +5C
- U3 pad 6: /A0 -> Net-(R22-Pad2)
- U3 pad 7: +5V -> +5C
Routing:
- net +5C: track 0.00 -> 215.3 mm, vias 0 -> 15
- net +5V: track 213.1 -> 0.00 mm, vias 15 -> 0
- net /REFO: track 29.1 -> 73.6 mm, vias 2 -> 3
- net Net-(C3-Pad1): track 55.0 -> 20.1 mm, vias 0 -> 2
- net /TP2: track 68.1 -> 90.8 mm, vias 2 -> 4
- net GND: track 712.8 -> 692.2 mm, vias 126 -> 128
- net /TP1: track 59.5 -> 79.8 mm, vias 0 -> 2
- net Net-(C3-Pad2): track 12.0 -> 0.00 mm
- net Net-(C13-Pad1): track 0.00 -> 9.60 mm
- net Net-(C2-Pad2): track 0.00 -> 9.58 mm
- net Net-(C2-Pad1): track 7.86 -> 0.00 mm
- net Net-(R22-Pad2): track 0.00 -> 5.61 mm
- net (no net): track 4.90 -> 0.00 mm, vias 3 -> 0
- net Net-(R20-Pad2): track 0.00 -> 4.70 mm
- net /A0: track 67.9 -> 67.2 mm, vias 4 -> 2
- added copper zone on B.Cu, net +5C
- removed copper zone on B.Cu, net +5V
Other:
- board text added: "v0.5"
- board text removed: "v0.4"

Commit message: update
Other:
- board text added: "V0.5"
Changed lines of the file:
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@@
     (links 156)
     (no_connects 0)
-    (area 49.924999 49.924999 150.075001 100.075001)
+    (area 47.6808 47.625 152.43256 102.075)
     (thickness 1.6)
-    (drawings 40)
+    (drawings 41)
     (tracks 1515)
     (zones 0)
@@
     )
   )
+  (gr_text V0.5 (at 54.75 98.25) (layer B.SilkS)
+    (effects (font (size 1 1) (thickness 0.15)) (justify mirror))
+  )
   (gr_text v0.5 (at 103.7 88.3) (layer F.SilkS)
