File: hardware/USBcablecracker.kicad_pcb (KiCad board)
At the start: 2 copper layers, 100 x 50 mm, 57 parts, among them P1 USB_A, P10 USB_A, P11 USB_B, P12 CONN_01X09, P2 CONN_01X02, P3 USB_B-Micro, P6 CONN_01X09, P7 USB_B-Mini, P8 USB_B-Micro-3.0, P9 USB_TYPEC-S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

Commit message: update
Parts:
- removed G***: LOGO, USBcablecracker:donotcare
Other:
- board text removed: "SZDIY COMMUNITY 2009.4.19-2017.4.19"

Commit message: update
Parts:
- added G***: LOGO, USBcablecracker:szdiy_logo, B.Cu at (78.8, 64.8)
Other:
- board text added: "USBcablecracker"
- board text added: "V1.0"
- board text removed: "V0.5"
